File: kicad/486SandwichSocketBlaster.kicad_pcb (KiCad board)
At the start: 2 copper layers, 49.2 x 52.2 mm, 30 parts, among them J1 Conn_02x11_Odd_Even, J10 Conn_01x16_Pin, J11 Conn_01x16_Pin, J2 Conn_02x11_Odd_Even, J3 Conn_02x06_Odd_Even, J4 Conn_01x18_Pin, J7 Conn_02x06_Odd_Even, J9 Conn_01x19_Pin, U3 VoltageRegulator

Commit message: Rev.0.2
Connections:
- net STPCLK_PIN renamed STPCLK_JMP
Other:
- board text added: "2x(DX4) 4x(5x86)"
- board text added: "486 Sandwich Socket Blaster rev.0.2"
- board text added: "Mobo"
- board text added: "PIN"
- board text added: "WB/WT"
- board text added: "rev.0.2"
- board text removed: "486 Sandwich Socket Blaster rev.0.1"
- board text removed: "CPUCLK"
- board text removed: "HOLD"
- board text removed: "User"
- board text removed: "rev.0.1"
