File: kicad/486SandwichSocketBlaster.kicad_sch (KiCad schematic)
At the start: 30 parts, among them J1 Conn_02x11_Odd_Even, J10 Conn_01x16_Pin, J11 Conn_01x16_Pin, J2 Conn_02x11_Odd_Even, J3 Conn_02x06_Odd_Even, J4 Conn_01x18_Pin, J7 Conn_02x06_Odd_Even, J9 Conn_01x19_Pin, U3 VoltageRegulator

Commit message: Rev.0.2
Connections:
- net STPCLK_PIN renamed STPCLK_JMP
Changed lines of the file:
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@@
   (title_block
     (title "486SandwichSocketBlaster")
-    (date "2024-10-06")
-    (rev "0.1")
+    (date "2024-10-19")
+    (rev "0.2")
     (company "ScrapComputing")
   )
@@
     )
   )
-  (global_label "STPCLK_PIN" (shape input) (at 190.5 388.62 90)
+  (global_label "STPCLK_JMP" (shape input) (at 190.5 388.62 90)
     (effects (font (size 1.27 1.27)) (justify left))
     (property "Intersheetrefs" "${INTERSHEET_REFS}" (at 190.5 388.62 0)
@@
     )
   )
-  (global_label "STPCLK_PIN" (shape input) (at 172.72 391.16 90) (fields_autoplaced)
-    (effects (font (size 1.27 1.27)) (justify left))
-    (property "Intersheetrefs" "${INTERSHEET_REFS}" (at 172.72 377.6409 90)
+  (global_label "STPCLK_JMP" (shape input) (at 172.72 391.16 90) (fields_autoplaced)
+    (effects (font (size 1.27 1.27)) (justify left))
+    (property "Intersheetrefs" "${INTERSHEET_REFS}" (at 172.72 377.1572 90)
       (effects (font (size 1.27 1.27)) (justify left) hide)
     )
@@
     )
   )
-  (global_label "STPCLK_PIN" (shape input) (at 177.8 354.33 0) (fields_autoplaced)
-    (effects (font (size 1.27 1.27)) (justify left))
-    (property "Intersheetrefs" "${INTERSHEET_REFS}" (at 191.3191 354.33 0)
+  (global_label "STPCLK_JMP" (shape input) (at 177.8 354.33 0) (fields_autoplaced)
+    (effects (font (size 1.27 1.27)) (justify left))
+    (property "Intersheetrefs" "${INTERSHEET_REFS}" (at 191.8028 354.33 0)
       (effects (font (size 1.27 1.27)) (justify left) hide)
     )
